File: Strain Gauge POC Board V1/Double Bridge 1.kicad_sch (KiCad schematic)
At the start: 49 parts, among them J301 Barrel_Jack, J302 502352-0210, U301 INA333xxDGK, U302 INA333xxDGK, U303 ADS1113IDGSR

Commit message: Working now
Parts:
- removed J301: Barrel_Jack, Connector_BarrelJack:BarrelJack_CUI_PJ-063AH_Horizontal, symbol Connector:Barrel_Jack
- C301, C302, C305, C306: Mfr PN CC0805KKX5R8BB106 -> GMC21X5R226M16NT
- C303, C304, C307: footprint Capacitor_SMD:C_0603_1608Metric -> ulib_Capacitor_SMD:C_0805_2012Metric; Mfr PN C0603C104J4RACTU -> GMC21X7R225K16NT; Package 0603 -> 0805; Voltage 50V -> 16V
- R304, R305, R308, R309, R314, R315, R316, R317, R318, R319, R320, R321, R324, R325: footprint ulib_Resistors_SMD:R_0603_1608Metric -> ulib_Resistors_SMD:R_1206_3216Metric; Mfr PN CRG0603F1K0 -> ESR18EZPJ102; Package 0603 -> 1206; Power 1/10W -> 1/2W; Tolerance 1% -> 5%
- R306, R307: footprint ulib_Resistors_SMD:R_0603_1608Metric -> ulib_Resistors_SMD:R_1206_3216Metric; Mfr PN RT0603BRC07500RL -> ESR18EZPJ102; Package 0603 -> 1206; Power 1/10W -> 1/2W; Tolerance 0.1% -> 5%
- R312, R313: footprint ulib_Resistors_SMD:R_0603_1608Metric -> ulib_Resistors_SMD:R_1206_3216Metric; Mfr PN RC0603FR-072K05L -> ESR18EZPJ102; Package 0603 -> 1206; Power 1/10W -> 1/2W; Tolerance 1% -> 5%
- R322, R323: footprint ulib_Resistors_SMD:R_0603_1608Metric -> ulib_Resistors_SMD:R_1206_3216Metric; Mfr PN RC0603JR-074K7L -> ESR18EZPJ102; Package 0603 -> 1206; Power 1/10W -> 1/2W

Commit message: dev
Parts:
- renumbered J302 to J301
Changed lines of the file:
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@@
 		(dnp no)
 		(fields_autoplaced yes)
-		(property "Reference" "J302"
+		(property "Reference" "J301"
 			(at 538.48 186.0549 90)
 			(effects
@@
 			(project "Strain Gauge POC Board V1"
 				(path "/86d41315-8564-4bca-9150-9edda69acf24/fe881be6-80bd-426d-a3d6-be163c7c4112"
-					(reference "J302")
+					(reference "J301")
 					(unit 1)
 				)
