File: Strain Gauge POC Board V1/Strain Gauge POC Board V1.kicad_sch (KiCad schematic)
At the start: 0 parts

Commit message: dev
Parts:
- added C101, C103: 10u, ulib_Capacitor_SMD:C_0805_2012Metric, symbol Capacitor 12V Picogrid:22u
- added C102, C104: 100n, ulib_Capacitor_SMD:C_0603_1608Metric, symbol ulib_Capacitor_SMD_250V:470p
- added FID101, FID102, FID103, FID104: Fiducial, ulib_Mechanical:Fiducial_0.5mm_Mask1mm, symbol ulib_Mounting_Holes:Fiducial
- added J101, J102: 502352-0210, ulib_Connectors_DuraClik:Molex_DuraClik_5023520210_1x02_MP_P2.00mm_Right_Angle, symbol ulib_Connectors_DuraClik:502352-0210
- added R101, R103, R106: 0, ulib_Resistors_SMD:R_0603_1608Metric, symbol ulib_Resistor_SMD_0.1W:0
- added R102, R105, R108, R109, R111, R112, R115, R116: 1k, ulib_Resistors_SMD:R_0603_1608Metric, symbol ulib_Resistor_SMD_0.1W:0
- added R104: 500, ulib_Resistors_SMD:R_0603_1608Metric, symbol ulib_Resistor_SMD_0.1W:0
- added R107: 2k05, ulib_Resistors_SMD:R_0603_1608Metric, symbol ulib_Resistor_SMD_0.1W:0
- added R110: 100R, ulib_Resistors_SMD:R_0603_1608Metric, symbol ulib_Resistor_SMD_0.1W:0
- added R113, R114: 4k7, ulib_Resistors_SMD:R_0603_1608Metric, symbol ulib_Resistor_SMD_0.1W:0
- added TP101, TP102: TestPoint, TestPoint:TestPoint_THTPad_D2.0mm_Drill1.0mm, symbol Connector:TestPoint
- added TP103, TP104: TestPoint, TestPoint:TestPoint_THTPad_D3.0mm_Drill1.5mm, symbol Connector:TestPoint
- added TP105, TP106: TestPoint, TestPoint:TestPoint_THTPad_D4.0mm_Drill2.0mm, symbol Connector:TestPoint
- added U101, U102, U103, U104: ~, ulib_Mechanical:MountingHole_3.2mm_M2_Pad_Via, symbol ulib_Mounting_Holes:M2 Pad
- added U105, U106, U107, U108: ~, TestPoint:TestPoint_Pad_D0.15mm, symbol ulib_TestPoints:Pad_0.15mm
- added U109: INA333xxDGK, Package_SO:VSSOP-8_3x3mm_P0.65mm, symbol Amplifier_Instrumentation:INA333xxDGK
- added U110: ADS1113IDGSR, ulib_Package_SO:SOP50P490X110-10N, symbol ulib_ADC_12b_16ch:ADS1113IDGSR
Connections:
- new net: R102.2, R104.1, R105.2, R106.2, U105.1, U106.1, U107.1, U108.1, U109.2 (-), U109.3 (+)
- new net: C103.1 (+), R106.1, R110.1, U110.4 (AIN0)
- new net: R110.2, U109.6
- new net: R103.2, U110.5 (AIN1)
- new net: C101.1 (+), R101.1, R102.1, R105.1
- new net: R111.1, R112.2, R115.2, R116.2, U110.1 (ADDR)
- new net: R107.1, U109.1 (Rg)
- new net: R107.2, U109.8 (Rg)
- new net: J102.2, R114.2, R115.1, U110.10 (SCL)
- new net: J102.1, R112.1, R113.2, U110.9 (SDA)
- new net +1V65a: R108.2, R109.1, U109.5 (Ref)
- new net +3V3a: C102.1 (+), C104.1 (+), J101.1, R101.2, R108.1, R113.1, R114.1, R116.1, TP101.1, TP103.1, TP105.1, U109.7 (V+), U110.8 (VDD)
- new net GND: C101.2 (-), C102.2 (-), C103.2 (-), C104.2 (-), J101.2, R104.2, R109.2, R111.2, TP102.1, TP104.1, TP106.1, U101.MP, U102.MP, U103.MP, U104.MP, U109.4 (V-), U110.3 (GND)
Other:
- removed sheet Double Bridge 1
- removed sheet Single Bridge 1
- note added: "1.1V nominal for each bridge node when strain gauge at rest"
- note added: "1.5mm plated holes"
- note added: "1mm plated holes"
- note added: "2mm plated holes"
- note added: "ADDR Address table"
- note added: "Compression Serpentine 1"
- note added: "Gain configurable 1-1000 G=1+(50k/R_G) for R_G=2.05k, G=50"
- note added: "Power Connectors suitable for dev board only"
- note added: "Strain Serpentine 1"
- note added: "f_c = 160Hz"
- note added: "f_c = TBD This filter is likely unnecessary and will only serve to drive up input impedance"
- note added: "minimize space between filter and ADC"
- note added: "minimize space between filter and wheatstone bridge"
- note added: "place right next to wheatstone output to minimize stub length"

Commit message: bulk of first draft done
Parts:
- removed C101, C103: 10u, ulib_Capacitor_SMD:C_0805_2012Metric, symbol Capacitor 12V Picogrid:22u
- removed C102, C104: 100n, ulib_Capacitor_SMD:C_0603_1608Metric, symbol ulib_Capacitor_SMD_250V:470p
- removed FID101, FID102, FID103, FID104: Fiducial, ulib_Mechanical:Fiducial_0.5mm_Mask1mm, symbol ulib_Mounting_Holes:Fiducial
- removed J101, J102: 502352-0210, ulib_Connectors_DuraClik:Molex_DuraClik_5023520210_1x02_MP_P2.00mm_Right_Angle, symbol ulib_Connectors_DuraClik:502352-0210
- removed R101, R103, R106: 0, ulib_Resistors_SMD:R_0603_1608Metric, symbol ulib_Resistor_SMD_0.1W:0
- removed R102, R105, R108, R109, R111, R112, R115, R116: 1k, ulib_Resistors_SMD:R_0603_1608Metric, symbol ulib_Resistor_SMD_0.1W:0
- removed R104: 500, ulib_Resistors_SMD:R_0603_1608Metric, symbol ulib_Resistor_SMD_0.1W:0
- removed R107: 2k05, ulib_Resistors_SMD:R_0603_1608Metric, symbol ulib_Resistor_SMD_0.1W:0
- removed R110: 100R, ulib_Resistors_SMD:R_0603_1608Metric, symbol ulib_Resistor_SMD_0.1W:0
- removed R113, R114: 4k7, ulib_Resistors_SMD:R_0603_1608Metric, symbol ulib_Resistor_SMD_0.1W:0
- removed TP101, TP102: TestPoint, TestPoint:TestPoint_THTPad_D2.0mm_Drill1.0mm, symbol Connector:TestPoint
- removed TP103, TP104: TestPoint, TestPoint:TestPoint_THTPad_D3.0mm_Drill1.5mm, symbol Connector:TestPoint
- removed TP105, TP106: TestPoint, TestPoint:TestPoint_THTPad_D4.0mm_Drill2.0mm, symbol Connector:TestPoint
- removed U101, U102, U103, U104: ~, ulib_Mechanical:MountingHole_3.2mm_M2_Pad_Via, symbol ulib_Mounting_Holes:M2 Pad
- removed U105, U106, U107, U108: ~, TestPoint:TestPoint_Pad_D0.15mm, symbol ulib_TestPoints:Pad_0.15mm
- removed U109: INA333xxDGK, Package_SO:VSSOP-8_3x3mm_P0.65mm, symbol Amplifier_Instrumentation:INA333xxDGK
- removed U110: ADS1113IDGSR, ulib_Package_SO:SOP50P490X110-10N, symbol ulib_ADC_12b_16ch:ADS1113IDGSR
Other:
- added sheet Single Bridge 1 (Single Bridge 1.kicad_sch)
- note removed: "1.1V nominal for each bridge node when strain gauge at rest"
- note removed: "1.5mm plated holes"
- note removed: "1mm plated holes"
- note removed: "2mm plated holes"
- note removed: "ADDR Address table"
- note removed: "Compression Serpentine 1"
- note removed: "Gain configurable 1-1000 G=1+(50k/R_G) for R_G=2.05k, G=50"
- note removed: "Power Connectors suitable for dev board only"
- note removed: "Strain Serpentine 1"
- note removed: "f_c = 160Hz"
- note removed: "f_c = TBD This filter is likely unnecessary and will only serve to drive up input impedance"
- note removed: "minimize space between filter and ADC"
- note removed: "minimize space between filter and wheatstone bridge"
- note removed: "place right next to wheatstone output to minimize stub length"
