File: Strain Gauge POC Board V1/Strain Gauge POC Board V1.kicad_pcb (KiCad board)
At the start: 4 copper layers, 70.7 x 19 mm, 2 parts

Commit message: Working now
Parts:
- added C201: 10u, ulib_Capacitor_SMD:C_0805_2012Metric, F.Cu at (171.3, 104.9)
- added C203: 10u, ulib_Capacitor_SMD:C_0805_2012Metric, F.Cu at (166.9, 99.3)
- added C204: 100n, ulib_Capacitor_SMD:C_0603_1608Metric, F.Cu at (168.7, 99.1)
- added C205: 100n, ulib_Capacitor_SMD:C_0603_1608Metric, F.Cu at (158.1, 95.9)
- added C301: 10u, ulib_Capacitor_SMD:C_0805_2012Metric, F.Cu at (-26.8, 18.1)
- added C302: 10u, ulib_Capacitor_SMD:C_0805_2012Metric, F.Cu at (-26.8, 21.1)
- added C303: 100n, ulib_Capacitor_SMD:C_0805_2012Metric, F.Cu at (-5.02, 29.6)
- added C304: 100n, ulib_Capacitor_SMD:C_0805_2012Metric, F.Cu at (-5.02, 32.1)
- added C305: 10u, ulib_Capacitor_SMD:C_0805_2012Metric, F.Cu at (-26.8, 24.2)
- added C306: 10u, ulib_Capacitor_SMD:C_0805_2012Metric, F.Cu at (-26.8, 27.2)
- added C307: 100n, ulib_Capacitor_SMD:C_0805_2012Metric, F.Cu at (-5.02, 34.6)
- added FID201: Fiducial, ulib_Mechanical:Fiducial_0.5mm_Mask1mm, F.Cu at (149.6, 110.7)
- added FID202: Fiducial, ulib_Mechanical:Fiducial_0.5mm_Mask1mm, F.Cu at (145.0, 111.0)
- added FID301: Fiducial, ulib_Mechanical:Fiducial_0.5mm_Mask1mm, F.Cu at (-1.74, 29.6)
- added FID302: Fiducial, ulib_Mechanical:Fiducial_0.5mm_Mask1mm, F.Cu at (-1.74, 32.2)
- added H301: M3-PAD, ulib_Mechanical:MountingHole_3.2mm_M3_Pad_Via, F.Cu at (-33.0, 2.67)
- added H302: M3-PAD, ulib_Mechanical:MountingHole_3.2mm_M3_Pad_Via, F.Cu at (-33.0, 10.6)
- added H303: M3-PAD, ulib_Mechanical:MountingHole_3.2mm_M3_Pad_Via, F.Cu at (-33.0, 18.6)
- added H304: M3-PAD, ulib_Mechanical:MountingHole_3.2mm_M3_Pad_Via, F.Cu at (-33.0, 26.5)
- added J202: 502352-0210, ulib_Connectors_DuraClik:Molex_DuraClik_5023520210_1x02_MP_P2.00mm_Right_Angle, F.Cu at (135.4, 92.4)
- added J203: 502352-0210, ulib_Connectors_DuraClik:Molex_DuraClik_5023520210_1x02_MP_P2.00mm_Right_Angle, F.Cu at (135.5, 104.9)
- added J302: 502352-0210, ulib_Connectors_DuraClik:Molex_DuraClik_5023520210_1x02_MP_P2.00mm_Right_Angle, F.Cu at (-12.9, 22.2)
- added R201: 0, ulib_Resistors_SMD:R_0603_1608Metric, F.Cu at (171.5, 103.1)
- added R202: 0, ulib_Resistors_SMD:R_0603_1608Metric, F.Cu at (174.5, 91.0)
- added R203: 1k, ulib_Resistors_SMD:R_0603_1608Metric, F.Cu at (174.1, 103.9)
- added R204: 4k7, ulib_Resistors_SMD:R_0603_1608Metric, F.Cu at (142.5, 101.6)
- added R205: 1k, ulib_Resistors_SMD:R_0603_1608Metric, F.Cu at (174.8, 95.2)
- added R206: 0, ulib_Resistors_SMD:R_0603_1608Metric, F.Cu at (172.1, 106.8)
- added R207: 100R, ulib_Resistors_SMD:R_0603_1608Metric, F.Cu at (167.0, 96.8)
- added R208: 1k, ulib_Resistors_SMD:R_0603_1608Metric, F.Cu at (168.7, 94.0)
- added R209: 1k, ulib_Resistors_SMD:R_0603_1608Metric, F.Cu at (170.4, 94.0)
- added R210: 4k7, ulib_Resistors_SMD:R_0603_1608Metric, F.Cu at (142.5, 106.8)
- added R211: 1k, ulib_Resistors_SMD:R_0603_1608Metric, F.Cu at (164.3, 100.8)
- added R212: 1k, ulib_Resistors_SMD:R_0603_1608Metric, F.Cu at (161.0, 100.8)
- added R213: 1k, ulib_Resistors_SMD:R_0603_1608Metric, F.Cu at (159.4, 100.8)
- added R214: 1k, ulib_Resistors_SMD:R_0603_1608Metric, F.Cu at (162.7, 100.8)
- added R217: 500, ulib_Resistors_SMD:R_0603_1608Metric, F.Cu at (174.0, 93.4)
- added R218: 2k05, ulib_Resistors_SMD:R_0603_1608Metric, F.Cu at (173.0, 100.8)
- added R301: 0, ulib_Resistors_SMD:R_0603_1608Metric, F.Cu at (-26.9, -0.03)
- added R302: 0, ulib_Resistors_SMD:R_0603_1608Metric, F.Cu at (-26.9, 2.52)
- added R303: 0, ulib_Resistors_SMD:R_0603_1608Metric, F.Cu at (-26.9, 5.08)
- added R304: 1k, ulib_Resistors_SMD:R_1206_3216Metric, F.Cu at (-26.9, 7.63)
- added R305: 1k, ulib_Resistors_SMD:R_1206_3216Metric, F.Cu at (-26.9, 10.2)
- added R306: 500R, ulib_Resistors_SMD:R_1206_3216Metric, F.Cu at (-26.9, 12.7)
- added R307: 500R, ulib_Resistors_SMD:R_1206_3216Metric, F.Cu at (-26.9, 15.3)
- added R308: 1k, ulib_Resistors_SMD:R_1206_3216Metric, F.Cu at (-22.8, -0.03)
- added R309: 1k, ulib_Resistors_SMD:R_1206_3216Metric, F.Cu at (-22.8, 2.52)
- added R310: 0, ulib_Resistors_SMD:R_0603_1608Metric, F.Cu at (-22.8, 5.08)
- added R311: 0, ulib_Resistors_SMD:R_0603_1608Metric, F.Cu at (-22.8, 7.63)
- added R312: 2k05, ulib_Resistors_SMD:R_1206_3216Metric, F.Cu at (-22.8, 10.2)
- added R313: 2k05, ulib_Resistors_SMD:R_1206_3216Metric, F.Cu at (-22.8, 12.7)
- added R314: 1k, ulib_Resistors_SMD:R_1206_3216Metric, F.Cu at (-22.8, 15.3)
- added R315: 1k, ulib_Resistors_SMD:R_1206_3216Metric, F.Cu at (-18.6, -0.03)
- added R316: 1k, ulib_Resistors_SMD:R_1206_3216Metric, F.Cu at (-18.6, 2.52)
- added R317: 1k, ulib_Resistors_SMD:R_1206_3216Metric, F.Cu at (-18.6, 5.08)
- added R318: 100R, ulib_Resistors_SMD:R_1206_3216Metric, F.Cu at (-18.6, 7.63)
- added R319: 100R, ulib_Resistors_SMD:R_1206_3216Metric, F.Cu at (-18.6, 10.2)
- added R320: 1k, ulib_Resistors_SMD:R_1206_3216Metric, F.Cu at (-18.6, 12.7)
- added R321: 1k, ulib_Resistors_SMD:R_1206_3216Metric, F.Cu at (-18.6, 15.3)
- added R322: 4k7, ulib_Resistors_SMD:R_1206_3216Metric, F.Cu at (-14.5, -0.03)
- added R323: 4k7, ulib_Resistors_SMD:R_1206_3216Metric, F.Cu at (-14.5, 2.52)
- added R324: 1k, ulib_Resistors_SMD:R_1206_3216Metric, F.Cu at (-14.5, 5.08)
- added R325: 1k, ulib_Resistors_SMD:R_1206_3216Metric, F.Cu at (-14.5, 7.63)
- added TP201: TestPoint, TestPoint:TestPoint_THTPad_D2.0mm_Drill1.0mm, F.Cu at (170.2, 88.9)
- added TP202: TestPoint, TestPoint:TestPoint_THTPad_D2.0mm_Drill1.0mm, F.Cu at (170.2, 109.5)
- added TP203: TestPoint, TestPoint:TestPoint_THTPad_D3.0mm_Drill1.5mm, F.Cu at (163.8, 88.9)
- added TP204: TestPoint, TestPoint:TestPoint_THTPad_D3.0mm_Drill1.5mm, F.Cu at (163.8, 109.5)
- added TP205: TestPoint, TestPoint:TestPoint_THTPad_D4.0mm_Drill2.0mm, F.Cu at (157.5, 88.9)
- added TP206: TestPoint, TestPoint:TestPoint_THTPad_D4.0mm_Drill2.0mm, F.Cu at (157.5, 109.5)
- added TP301: TestPoint, TestPoint:TestPoint_THTPad_D2.0mm_Drill1.0mm, F.Cu at (-9.05, 30.4)
- added TP302: TestPoint, TestPoint:TestPoint_THTPad_D2.0mm_Drill1.0mm, F.Cu at (-9.05, 34.4)
- added TP303: TestPoint, TestPoint:TestPoint_THTPad_D3.0mm_Drill1.5mm, F.Cu at (-4.75, 19.1)
- added TP304: TestPoint, TestPoint:TestPoint_THTPad_D3.0mm_Drill1.5mm, F.Cu at (-4.75, 24.1)
- added TP305: TestPoint, TestPoint:TestPoint_THTPad_D4.0mm_Drill2.0mm, F.Cu at (-21.5, 19.6)
- added TP306: TestPoint, TestPoint:TestPoint_THTPad_D4.0mm_Drill2.0mm, F.Cu at (-21.5, 25.6)
- added U201: INA333xxDGK, Package_SO:VSSOP-8_3x3mm_P0.65mm, F.Cu at (172.9, 98.0)
- added U202: ADS1113IDGSR, ulib_Package_SO:SOP50P490X110-10N, F.Cu at (162.2, 97.3)
- added U205: ~, TestPoint:TestPoint_Pad_D0.15mm, F.Cu at (176.8, 99.8)
- added U206: ~, TestPoint:TestPoint_Pad_D0.15mm, F.Cu at (177.5, 95.8)
- added U207: ~, TestPoint:TestPoint_Pad_D0.15mm, F.Cu at (176.5, 97.4)
- added U208: ~, TestPoint:TestPoint_Pad_D0.15mm, F.Cu at (176.5, 94.7)
- added U209: ~, ulib_Mechanical:MountingHole_3.2mm_M2_Pad_Via, F.Cu at (148.3, 91.6)
- added U210: ~, ulib_Mechanical:MountingHole_3.2mm_M2_Pad_Via, F.Cu at (148.3, 104.6)
- added U301: INA333xxDGK, Package_SO:VSSOP-8_3x3mm_P0.65mm, F.Cu at (-14.8, 30.7)
- added U302: INA333xxDGK, Package_SO:VSSOP-8_3x3mm_P0.65mm, F.Cu at (-14.8, 35.4)
- added U303: ADS1113IDGSR, ulib_Package_SO:SOP50P490X110-10N, F.Cu at (-32.7, 32.8)
- moved U203 32.7 mm to (178.2, 91.6)
- moved U204 32.7 mm to (178.2, 104.6)
Routing:
- net Net-(U201-+): track 0.00 -> 125.1 mm, vias 0 -> 2
- net +3V3a: track 0.00 -> 93.4 mm, vias 0 -> 5
- net Net-(U202-SDA): track 0.00 -> 28.6 mm
- net Net-(U202-SCL): track 0.00 -> 26.0 mm
- net GND: track 0.00 -> 24.3 mm, vias 0 -> 9
- net Net-(C203-+): track 0.00 -> 16.3 mm
- net Net-(U202-AIN1): track 0.00 -> 13.4 mm
- net Net-(C201-+): track 0.00 -> 12.7 mm
- net Net-(U202-ADDR): track 0.00 -> 8.94 mm
- net +1V65a: track 0.00 -> 4.17 mm
- net Net-(R207-Pad2): track 0.00 -> 3.35 mm
- net Net-(R218-Pad2): track 0.00 -> 3.09 mm
- net Net-(R218-Pad1): track 0.00 -> 2.90 mm
- added copper zone on In1.Cu, net GND
- added copper zone on In2.Cu, net GND
Other:
- board size 70.7 x 19 mm -> 75.6 x 31.5 mm
- board text added: "I2C"
- board text added: "PWR"

Commit message: dev
Parts:
- moved TP202 1.52 mm to (170.2, 111.0)
- moved TP204 1.52 mm to (163.8, 111.0)
- moved TP206 1.52 mm to (157.5, 111.0)
Routing:
- net +3V3a: track 93.4 -> 108.6 mm, vias 5 -> 6
- net GND: track 24.3 -> 25.0 mm, vias 9 -> 10
Other:
- board text added: "+3V3"
- board text added: "GND"
- board text removed: "PWR"
Changed lines of the file:
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@@
 		(tags "resistor")
 		(property "Reference" "R213"
-			(at 0 -1.27 90)
+			(at 2.7 -0.115 90)
 			(layer "F.SilkS" knockout)
 			(effects
@@
 		(tags "resistor")
 		(property "Reference" "R212"
-			(at 0 -1.27 90)
+			(at 2.7 -0.064 90)
 			(layer "F.SilkS" knockout)
 			(effects
@@
 	(footprint "TestPoint:TestPoint_THTPad_D3.0mm_Drill1.5mm"
 		(layer "F.Cu")
-		(at 163.83 109.474 180)
+		(at 163.83 110.998 180)
 		(descr "THT pad as test Point, diameter 3.0mm, hole diameter 1.5mm")
 		(tags "test point THT pad")
@@
 	(footprint "TestPoint:TestPoint_THTPad_D2.0mm_Drill1.0mm"
 		(layer "F.Cu")
-		(at 170.18 109.474 180)
+		(at 170.18 110.998 180)
 		(descr "THT pad as test Point, diameter 2.0mm, hole diameter 1.0mm")
 		(tags "test point THT pad")
@@
 		(tags "resistor")
 		(property "Reference" "R211"
-			(at 0 -1.27 90)
+			(at -2.7 -1.738 90)
 			(layer "F.SilkS" knockout)
 			(effects
@@
 		(tags "resistor")
 		(property "Reference" "R214"
-			(at 0 -1.27 90)
+			(at 2.7 -1.713 90)
 			(layer "F.SilkS" knockout)
 			(effects
@@
 	(footprint "TestPoint:TestPoint_THTPad_D4.0mm_Drill2.0mm"
 		(layer "F.Cu")
-		(at 157.48 109.474 180)
+		(at 157.48 110.998 180)
 		(descr "THT pad as test Point, diameter 4.0mm, hole diameter 2.0mm")
 		(tags "test point THT pad")
@@
 		(tags "capacitor")
 		(property "Reference" "C205"
-			(at 0 -1.27 90)
+			(at 0.085 -1.415 90)
 			(layer "F.SilkS" knockout)
 			(effects
@@
 	)
 	(gr_rect
+		(start 154.703984 107.736817)
+		(end 171.940016 114.046)
+		(stroke
+			(width 0.1)
+			(type default)
+		)
+		(fill no)
+		(layer "F.SilkS")
+	)
+	(gr_rect
+		(start 154.686 85.598)
+		(end 171.922032 91.907183)
+		(stroke
+			(width 0.1)
+			(type default)
+		)
+		(fill no)
+		(layer "F.SilkS")
+	)
+	(gr_rect
 		(start 178.164659 96.008806)
 		(end 183.784206 100.208406)
@@
 		(layer "Edge.Cuts")
 	)
-	(gr_text "PWR"
+	(gr_text "+3V3"
 		(at 127.601 90.186 270)
 		(layer "F.SilkS")
@@
 		)
 	)
+	(gr_text "GND"
+		(at 158.917984 107.438817 0)
+		(layer "F.SilkS")
+		(effects
+			(font
+				(size 1.5 1.5)
+				(thickness 0.3)
+				(bold yes)
+			)
+			(justify left bottom)
+		)
+	)
+	(gr_text "+3V3"
+		(at 158.9 85.3 0)
+		(layer "F.SilkS")
+		(effects
+			(font
+				(size 1.5 1.5)
+				(thickness 0.3)
+				(bold yes)
+			)
+			(justify left bottom)
+		)
+	)
 	(segment
 		(start 173.0099 101.4371)
@@
 	)
 	(segment
-		(start 163.83 109.474)
-		(end 170.18 109.474)
+		(start 163.83 110.998)
+		(end 170.18 110.998)
 		(width 1.016)
 		(layer "F.Cu")
@@
 	)
 	(segment
-		(start 157.48 109.474)
-		(end 163.83 109.474)
+		(start 157.48 110.998)
+		(end 163.83 110.998)
 		(width 1.016)
 		(layer "F.Cu")
@@
 	)
 	(segment
-		(start 173.228 93.431)
-		(end 173.228 92.161)
-		(width 0.14986)
+		(start 158.204 94.996)
+		(end 158.115 95.085)
+		(width 0.3048)
 		(layer "F.Cu")
 		(net 2)
 	)
 	(segment
-		(start 158.204 94.996)
-		(end 158.115 95.085)
-		(width 0.3048)
+		(start 163.322 97.282)
+		(end 163.068 97.282)
+		(width 0.199898)
 		(layer "F.Cu")
 		(net 2)
 	)
 	(segment
-		(start 175.006 97.028)
-		(end 173.736 97.028)
-		(width 0.3048)
+		(start 173.736 97.028)
+		(end 173.791 96.973)
+		(width 0.508)
 		(layer "F.Cu")
 		(net 2)
 	)
 	(segment
-		(start 163.322 97.282)
-		(end 163.068 97.282)
-		(width 0.199898)
+		(start 173.228 93.431)
+		(end 173.228 92.456)
+		(width 0.508)
 		(layer "F.Cu")
 		(net 2)
@@
 	)
 	(segment
+		(start 173.791 96.973)
+		(end 175.006 96.973)
+		(width 0.508)
+		(layer "F.Cu")
+		(net 2)
+	)
+	(segment
 		(start 166.878 100.203)
 		(end 166.878 101.092)
@@
 	)
 	(segment
+		(start 170.434 93.18)
+		(end 170.434 92.202)
+		(width 0.508)
+		(layer "F.Cu")
+		(net 2)
+	)
+	(segment
 		(start 170.35 104.902)
 		(end 169.672 104.902)
@@
 	)
 	(via
-		(at 173.228 92.161)
+		(at 173.228 92.456)
+		(size 0.6)
+		(drill 0.3)
+		(layers "F.Cu" "B.Cu")
+		(net 2)
+	)
+	(via
+		(at 170.434 92.202)
 		(size 0.6)
 		(drill 0.3)
@@
 	)
 	(segment
-		(start 167.259 93.345)
-		(end 168.491 93.345)
-		(width 0.3048)
+		(start 157.48 88.9)
+		(end 163.83 88.9)
+		(width 1.016)
 		(layer "F.Cu")
 		(net 3)
 	)
 	(segment
-		(start 157.48 88.9)
-		(end 163.83 88.9)
-		(width 1.016)
+		(start 168.491 93.345)
+		(end 168.656 93.18)
+		(width 0.508)
 		(layer "F.Cu")
 		(net 3)
@@
 	)
 	(segment
-		(start 168.491 93.345)
-		(end 168.656 93.18)
+		(start 170.751 98.298)
+		(end 170.781 98.328)
 		(width 0.3048)
 		(layer "F.Cu")
@@
 	)
 	(segment
-		(start 170.751 98.298)
-		(end 170.781 98.328)
-		(width 0.3048)
+		(start 167.259 93.345)
+		(end 168.491 93.345)
+		(width 0.508)
 		(layer "F.Cu")
 		(net 3)
@@
 	)
 	(segment
+		(start 142.494 108.966)
+		(end 142.494 107.595)
+		(width 1.016)
+		(layer "F.Cu")
+		(net 3)
+	)
+	(segment
+		(start 142.494 107.595)
+		(end 142.52 107.569)
+		(width 1.016)
+		(layer "F.Cu")
+		(net 3)
+	)
+	(segment
 		(start 161.544 97.282)
 		(end 160.029 97.282)
@@
 	)
 	(via
+		(at 142.494 108.966)
+		(size 0.6)
+		(drill 0.3)
+		(layers "F.Cu" "B.Cu")
+		(net 3)
+	)
+	(via
 		(at 172.212 98.298)
 		(size 0.6)
@@
 	)
 	(segment
+		(start 142.52 108.94)
+		(end 142.494 108.966)
+		(width 1.016)
+		(layer "B.Cu")
+		(net 3)
+	)
+	(segment
 		(start 144.78 96.012)
 		(end 144.018 95.25)
@@
 		(width 1.016)
 		(layer "B.Cu")
+		(net 3)
+	)
+	(segment
+		(start 142.52 95.25)
+		(end 142.52 108.94)
+		(width 1.016)
+		(layer "B.Cu")

Commit message: dev
Other:
- board text added: "+"
- board text added: "-"
Changed lines of the file:
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@@
 		(tags "resistor")
 		(property "Reference" "R206"
-			(at 0 -1.27 0)
+			(at 0.777 1.193 0)
 			(layer "F.SilkS" knockout)
 			(effects
@@
 		(tags "resistor")
 		(property "Reference" "R204"
-			(at 0 -1.27 90)
+			(at -0.962 -1.88 0)
 			(layer "F.SilkS" knockout)
 			(effects
@@
 		(tags "resistor")
 		(property "Reference" "R208"
-			(at -2.68 -0.044 90)
+			(at -2.08 0.356 0)
 			(layer "F.SilkS" knockout)
 			(effects
@@
 			(at 0 -2.398 0)
 			(layer "F.SilkS")
+			(hide yes)
 			(effects
 				(font
@@
 			(layer "F.CrtYd")
 		)
-		(fp_text user "${REFERENCE}"
-			(at 0 -2.4 0)
-			(layer "F.Fab")
-			(effects
-				(font
-					(size 1 1)
-					(thickness 0.15)
-				)
-			)
-		)
 		(pad "1" thru_hole circle
 			(at 0 0 180)
@@
 			(at 0 -2.398 0)
 			(layer "F.SilkS")
+			(hide yes)
 			(effects
 				(font
@@
 			(layer "F.CrtYd")
 		)
-		(fp_text user "${REFERENCE}"
-			(at 0 -2.4 0)
-			(layer "F.Fab")
-			(effects
-				(font
-					(size 1 1)
-					(thickness 0.15)
-				)
-			)
-		)
 		(pad "1" thru_hole circle
 			(at 0 0 180)
@@
 		(tags "resistor")
 		(property "Reference" "R217"
-			(at 0 -1.27 0)
+			(at -3.072 -1.169 0)
 			(layer "F.SilkS" knockout)
 			(effects
@@
 			(at 0 -1.998 0)
 			(layer "F.SilkS")
+			(hide yes)
 			(effects
 				(font
@@
 			(layer "F.CrtYd")
 		)
-		(fp_text user "${REFERENCE}"
-			(at 0 -2 0)
-			(layer "F.Fab")
-			(effects
-				(font
-					(size 1 1)
-					(thickness 0.15)
-				)
-			)
-		)
 		(pad "1" thru_hole circle
 			(at 0 0 180)
@@
 		(tags "resistor")
 		(property "Reference" "R210"
-			(at 0 -1.27 90)
+			(at 0.969 1.88 0)
 			(layer "F.SilkS" knockout)
 			(effects
@@
 		)
 		(fp_text user "${REFERENCE}"
-			(at 0 2.54 90)
+			(at 0 0 90)
 			(layer "F.Fab")
 			(effects
@@
 			(at 0 -1.998 0)
 			(layer "F.SilkS")
+			(hide yes)
 			(effects
 				(font
@@
 			(layer "F.CrtYd")
 		)
-		(fp_text user "${REFERENCE}"
-			(at 0 -2 0)
-			(layer "F.Fab")
-			(effects
-				(font
-					(size 1 1)
-					(thickness 0.15)
-				)
-			)
-		)
 		(pad "1" thru_hole circle
 			(at 0 0 180)
@@
 		(tags "test point SMD pad")
 		(property "Reference" "U206"
-			(at 0 -1.448 0)
+			(at 6.354 -1.758 0)
 			(layer "F.SilkS")
 			(effects
@@
 		(attr exclude_from_pos_files)
 		(fp_text user "${REFERENCE}"
-			(at 0 -1.45 0)
+			(at 6.354 -1.76 0)
 			(layer "F.Fab")
 			(effects
@@
 			(at 0 -2.898 0)
 			(layer "F.SilkS")
+			(hide yes)
 			(effects
 				(font
@@
 			(layer "F.CrtYd")
 		)
-		(fp_text user "${REFERENCE}"
-			(at 0 -2.9 0)
-			(layer "F.Fab")
-			(effects
-				(font
-					(size 1 1)
-					(thickness 0.15)
-				)
-			)
-		)
 		(pad "1" thru_hole circle
 			(at 0 0 180)
@@
 		(tags "resistor")
 		(property "Reference" "R202"
-			(at 0 -1.27 90)
+			(at 0.121 -1.898 180)
 			(layer "F.SilkS" knockout)
 			(effects
@@
 		(tags "resistor")
 		(property "Reference" "R209"
-			(at 2.68 0.066 90)
+			(at 2.08 0.266 180)
 			(layer "F.SilkS" knockout)
 			(effects
@@
 		(tags "connector Molex DuraClik side entry")
 		(property "Reference" "J202"
-			(at -3.683 4.191 90)
+			(at -4.676 4.518 0)
 			(unlocked yes)
 			(layer "F.SilkS" knockout)
@@
 		(tags "connector Molex DuraClik side entry")
 		(property "Reference" "J203"
-			(at -3.683 4.191 90)
+			(at -4.614 4.436 0)
 			(unlocked yes)
 			(layer "F.SilkS" knockout)
@@
 		(tags "test point SMD pad")
 		(property "Reference" "U207"
-			(at 0 -1.448 0)
+			(at 9.17 -0.68057 0)
 			(layer "F.SilkS")
 			(effects
@@
 		(attr exclude_from_pos_files)
 		(fp_text user "${REFERENCE}"
-			(at 0 -1.45 0)
+			(at 9.17 -0.68257 0)
 			(layer "F.Fab")
 			(effects
@@
 			(at 0 -2.898 0)
 			(layer "F.SilkS")
+			(hide yes)
 			(effects
 				(font
@@
 			(at 0 3.1 0)
 			(layer "F.Fab")
+			(hide yes)
 			(effects
 				(font
@@
 			(layer "F.CrtYd")
 		)
-		(fp_text user "${REFERENCE}"
-			(at 0 -2.9 0)
-			(layer "F.Fab")
-			(effects
-				(font
-					(size 1 1)
-					(thickness 0.15)
-				)
-			)
-		)
 		(pad "1" thru_hole circle
 			(at 0 0 180)
@@
 		(tags "resistor")
 		(property "Reference" "R205"
-			(at 0 -1.27 0)
+			(at -2.452 0 0)
 			(layer "F.SilkS" knockout)
 			(effects
@@
 		(layer "F.SilkS")
 		(effects
+			(font
+				(size 1.5 1.5)
+				(thickness 0.3)
+				(bold yes)
+			)
+			(justify left bottom)
+		)
+	)
+	(gr_text "-"
+		(at 141.332 94.8 180)
+		(layer "F.SilkS")
+		(effects
+			(font
+				(size 1.5 1.5)
+				(thickness 0.3)
+				(bold yes)
+			)
+			(justify left bottom)
+		)
+	)
+	(gr_text "+"
+		(at 139.3 90.6 0)
+		(layer "F.SilkS")
+		(effects

Commit message: dev
Parts:
- removed C301, C302, C305, C306: 10u, ulib_Capacitor_SMD:C_0805_2012Metric
- removed C303, C304, C307: 100n, ulib_Capacitor_SMD:C_0805_2012Metric
- removed FID201, FID202, FID301, FID302: Fiducial, ulib_Mechanical:Fiducial_0.5mm_Mask1mm
- removed H301, H302, H303, H304: M3-PAD, ulib_Mechanical:MountingHole_3.2mm_M3_Pad_Via
- removed J302: 502352-0210, ulib_Connectors_DuraClik:Molex_DuraClik_5023520210_1x02_MP_P2.00mm_Right_Angle
- removed R301, R302, R303, R310, R311: 0, ulib_Resistors_SMD:R_0603_1608Metric
- removed R304, R305, R308, R309, R314, R315, R316, R317, R320, R321, R324, R325: 1k, ulib_Resistors_SMD:R_1206_3216Metric
- removed R306, R307: 500R, ulib_Resistors_SMD:R_1206_3216Metric
- removed R312, R313: 2k05, ulib_Resistors_SMD:R_1206_3216Metric
- removed R318, R319: 100R, ulib_Resistors_SMD:R_1206_3216Metric
- removed R322, R323: 4k7, ulib_Resistors_SMD:R_1206_3216Metric
- removed TP301, TP302: TestPoint, TestPoint:TestPoint_THTPad_D2.0mm_Drill1.0mm
- removed TP303, TP304: TestPoint, TestPoint:TestPoint_THTPad_D3.0mm_Drill1.5mm
- removed TP305, TP306: TestPoint, TestPoint:TestPoint_THTPad_D4.0mm_Drill2.0mm
- removed U301, U302: INA333xxDGK, Package_SO:VSSOP-8_3x3mm_P0.65mm
- removed U303: ADS1113IDGSR, ulib_Package_SO:SOP50P490X110-10N
- added FID101: Fiducial, ulib_Mechanical:Fiducial_0.5mm_Mask1mm, F.Cu at (127.3, 88.9)
- added FID102: Fiducial, ulib_Mechanical:Fiducial_0.5mm_Mask1mm, F.Cu at (175.5, 81.8)
- added FID103: Fiducial, ulib_Mechanical:Fiducial_0.5mm_Mask1mm, F.Cu at (127.5, 111.5)
- added FID104: Fiducial, ulib_Mechanical:Fiducial_0.5mm_Mask1mm, F.Cu at (175.5, 111.3)
- added G***: LOGO, ulib_Logos:picogrid_logo, F.Cu at (140.0, 83.6)
- moved R208 0.80 mm to (167.9, 93.7)
- moved R209 0.80 mm to (169.7, 93.7)
- moved R206 0.42 mm to (171.7, 106.8)
- renumbered C204 to C202, C205 to C204, J202 to J201, J203 to J202, R203 to R202, R202 to R203, R217 to R204, R218 to R207, R207 to R210, R204 to R213, R210 to R214, R213 to R215, R214 to R216, U203 to U201, U204 to U202, U209 to U203, U210 to U204, U201 to U209, U202 to U210
Routing:
- net (no net): track 0.00 -> 14.0 mm
- net Net-(U210-AIN1): track 13.4 -> 0.00 mm
- net Net-(U209-+): track 125.1 -> 131.1 mm
- net +1V65a: track 4.17 -> 5.21 mm
Other:
- board size 75.6 x 31.5 mm -> 75.6 x 35.3 mm
- board text added: "M2"
- board text added: "SCL"
- board text added: "SDA"

Commit message: bulk of first draft done
Parts:
- removed FID101, FID102, FID103, FID104: Fiducial, ulib_Mechanical:Fiducial_0.5mm_Mask1mm
- added FID201: Fiducial, ulib_Mechanical:Fiducial_0.5mm_Mask1mm, F.Cu at (128.3, 91.9)
- added FID202: Fiducial, ulib_Mechanical:Fiducial_0.5mm_Mask1mm, F.Cu at (174.0, 86.9)
- added FID203: Fiducial, ulib_Mechanical:Fiducial_0.5mm_Mask1mm, F.Cu at (128.3, 111.5)
- added FID204: Fiducial, ulib_Mechanical:Fiducial_0.5mm_Mask1mm, F.Cu at (174.2, 111.5)
- moved J201 3.62 mm to (134.7, 96.0)
- moved J202 3.62 mm to (134.8, 108.4)
- moved R213 3.62 mm to (141.8, 105.1)
- moved R214 3.62 mm to (141.8, 110.3)
- moved G*** 3.57 mm to (140.2, 87.1)
Routing:
- net Net-(U210-AIN1): track 0.00 -> 14.9 mm
- net (no net): track 14.0 -> 0.00 mm
- net Net-(U210-SDA): track 28.6 -> 32.6 mm
- net Net-(U210-SCL): track 26.0 -> 29.8 mm
- net +3V3a: track 108.3 -> 110.0 mm, vias 6 -> 7
- net Net-(U209-+): track 131.1 -> 130.5 mm
Other:
- board size 75.6 x 35.3 mm -> 75.6 x 31.4 mm

Commit message: further dev
Routing:
- net +3V3a: track 110.0 -> 106.4 mm
Other:
- board text added: "Strain Gauge Test Board Date: 20250604 Designer: Clay Clemmer"

Commit message: almost finished first draft
Routing:
- net +3V3a: track 106.4 -> 105.0 mm
- net Net-(U210-SDA): track 32.6 -> 31.2 mm
- net Net-(U210-SCL): track 29.8 -> 28.9 mm
- net Net-(C201-+): track 12.7 -> 12.1 mm
