File: Strain Gauge POC Board V1/Strain Gauge POC Board V1.kicad_pcb (KiCad board)
At the start: 4 copper layers, 75.6 x 31.4 mm, 43 parts, among them J201 502352-0210, J202 502352-0210, U209 INA333xxDGK, U210 ADS1113IDGSR

Commit message: Ready for fab sans watermark
Parts:
- moved R214 18.0 mm to (156.2, 99.5)
- moved R213 14.6 mm to (153.9, 97.0)
- moved R211 1.30 mm to (164.4, 102.1)
- moved R215 1.30 mm to (159.4, 102.1), turned to 90 degrees
- moved R212 1.30 mm to (161.1, 102.1), turned to 90 degrees
- moved R216 1.30 mm to (162.7, 102.1), turned to 90 degrees
Connections:
- J202 pad 1: Net-(U210-SDA) -> ADC_I2C_SDA
- J202 pad 2: Net-(U210-SCL) -> ADC_I2C_SCL
- R203 pad 1: unconnected-(R203-Pad1) -> Net-(U209-+)
- R212 pad 1: Net-(U210-SDA) -> Net-(U210-ADDR)
- R212 pad 2: Net-(U210-ADDR) -> ADC_I2C_SDA
- R213 pad 2: Net-(U210-SDA) -> ADC_I2C_SDA
- R214 pad 2: Net-(U210-SCL) -> ADC_I2C_SCL
- R215 pad 1: Net-(U210-SCL) -> Net-(U210-ADDR)
- R215 pad 2: Net-(U210-ADDR) -> ADC_I2C_SCL
- R216 pad 1: +3V3a -> Net-(U210-ADDR)
- R216 pad 2: Net-(U210-ADDR) -> +3V3a
- U210 pad 10: Net-(U210-SCL) -> ADC_I2C_SCL
- U210 pad 9: Net-(U210-SDA) -> ADC_I2C_SDA
Routing:
- net ADC_I2C_SDA: track 0.00 -> 32.0 mm
- net ADC_I2C_SCL: track 0.00 -> 31.5 mm
- net Net-(U210-SDA): track 31.2 -> 0.00 mm
- net Net-(U210-SCL): track 28.9 -> 0.00 mm
- net +3V3a: track 105.0 -> 85.6 mm, vias 7 -> 5
- net GND: track 25.0 -> 22.8 mm, vias 10 -> 11
- net Net-(U210-ADDR): track 8.73 -> 10.6 mm
- net Net-(U209-+): track 130.5 -> 132.2 mm
Other:
- board text added: "3V3"
- board text added: "I2C Config Resistors"
- board text removed: "M2"
- board text removed: "Strain Gauge Test Board Date: 20250604 Designer: Clay Clemmer"
