File: Strain Gauge POC Board V1/Strain Gauge POC Board V1.kicad_pcb (KiCad board)
At the start: 4 copper layers, 75.6 x 31.4 mm, 43 parts, among them J201 502352-0210, J202 502352-0210, U209 INA333xxDGK, U210 ADS1113IDGSR

Commit message: dev
Routing:
- net ADC_I2C_SCL: track 31.5 -> 29.8 mm
- net ADC_I2C_SDA: track 32.0 -> 32.6 mm
Other:
- board text added: "${LAST_EDIT_DATE} ${VERSION} Rev. ${REV}"
- board text added: "${TITLE}"

Commit message: dev
Parts:
- added U201: ~, ulib_Mechanical:MountingHole_3.2mm_M2_Pad_Via, F.Cu at (171.8, 105.5)
- added U202: ~, ulib_Mechanical:MountingHole_3.2mm_M2_Pad_Via, F.Cu at (171.8, 119.2)
- moved U201 53.0 mm to (167.8, 39.7)
- moved C201 52.6 mm to (161.1, 53.3)
- moved C204 52.6 mm to (147.9, 44.3)
- moved FID203 52.6 mm to (118.1, 59.9)
- moved FID204 52.6 mm to (164.1, 59.9)
- moved G*** 52.6 mm to (130.0, 35.5)
- moved J201 52.6 mm to (124.5, 44.4)
- moved R203 52.6 mm to (164.3, 39.4)
- moved R205 52.6 mm to (164.6, 43.6)
- moved R206 52.6 mm to (161.5, 55.2)
- moved R210 52.6 mm to (156.8, 45.2)
- moved R213 52.6 mm to (143.7, 45.4)
- moved R214 52.6 mm to (146.0, 47.9)
- moved TP201 52.6 mm to (160.0, 37.3)
- moved TP202 52.6 mm to (160.0, 59.4)
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Other:
- board size 75.6 x 31.4 mm -> 109.8 x 97.3 mm
- board text added: "Widened channel between M2 and flexure to be exact mill bit dimensions of 0.068{dblquote} diameter"

Commit message: dev
Other:
- board size 109.8 x 97.3 mm -> 95.7 x 97.3 mm
- board text added: "widened flexure to gain 0.6mm width"
Changed lines of the file:
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@@
 	)
 	(gr_circle
-		(center 178.5874 101.6254)
-		(end 179.451 101.6254)
+		(center 183.642 82.042)
+		(end 184.5056 82.042)
 		(stroke
 			(width 0.1)
@@
 	)
 	(gr_arc
-		(start 208.03348 109.964808)
-		(mid 224.0534 112.6998)
-		(end 208.033488 115.434839)
+		(start 172.659977 116.835909)
+		(mid 172.274643 115.893896)
+		(end 173.009373 115.189594)
 		(stroke
 			(width 0.05)
@@
 		(layer "Edge.Cuts")
 	)
-	(gr_arc
-		(start 172.659977 116.835909)
-		(mid 172.274643 115.893896)
-		(end 173.009373 115.189594)
+	(gr_line
+		(start 181.9118 102.68275)
+		(end 208.429178 102.679803)
 		(stroke
 			(width 0.05)
@@
 	)
 	(gr_arc
+		(start 210.016678 120.511897)
+		(mid 209.551711 121.63443)
+		(end 208.429178 122.099397)
+		(stroke
+			(width 0.2)
+			(type default)
+		)
+		(layer "Edge.Cuts")
+	)
+	(gr_arc
 		(start 173.893495 43.791345)
 		(mid 173.711884 43.963672)
@@
 	)
 	(gr_arc
+		(start 208.429178 102.679803)
+		(mid 209.551711 103.14477)
+		(end 210.016678 104.267303)
+		(stroke
+			(width 0.2)
+			(type default)
+		)
+		(layer "Edge.Cuts")
+	)
+	(gr_arc
 		(start 173.575015 102.889606)
 		(mid 174.282107 103.182514)
@@
 		(layer "Edge.Cuts")
 	)
+	(gr_line
+		(start 181.759178 122.099397)
+		(end 181.759178 115.192553)
+		(stroke
+			(width 0.05)
+			(type solid)
+		)
+		(layer "Edge.Cuts")
+	)
 	(gr_arc
 		(start 170.094992 51.620551)
@@
 		(layer "Edge.Cuts")
 	)
-	(gr_arc
-		(start 208.033488 109.964813)
-		(mid 207.851877 110.13714)
-		(end 207.609488 110.199813)
+	(gr_line
+		(start 208.429178 122.099397)
+		(end 181.759178 122.099397)
 		(stroke
 			(width 0.05)
@@
 	)
 	(gr_line
+		(start 210.016678 120.511897)
+		(end 210.016678 104.267303)
+		(stroke
+			(width 0.2)
+			(type default)
+		)
+		(layer "Edge.Cuts")
+	)
+	(gr_circle
+		(center 184.890706 106.553303)
+		(end 187.640706 106.553303)
+		(stroke
+			(width 0.2)
+			(type default)
+		)
+		(fill no)
+		(layer "Edge.Cuts")
+	)
+	(gr_line
 		(start 168.523984 62.702739)
 		(end 115.275192 62.702739)
@@
 		(layer "Edge.Cuts")
 	)
+	(gr_circle
+		(center 195.516942 112.3896)
+		(end 199.288842 112.3896)
+		(stroke
+			(width 0.2)
+			(type default)
+		)
+		(fill no)
+		(layer "Edge.Cuts")
+	)
 	(gr_line
 		(start 170.524807 40.033851)
@@
 	)
 	(gr_line
+		(start 175.511254 63.252)
+		(end 193.511254 63.252)
+		(stroke
+			(width 0.05)
+			(type solid)
+		)
+		(layer "Edge.Cuts")
+	)
+	(gr_circle
+		(center 206.143178 118.225897)
+		(end 208.893178 118.225897)
+		(stroke
+			(width 0.2)
+			(type default)
+		)
+		(fill no)
+		(layer "Edge.Cuts")
+	)
+	(gr_line
 		(start 173.575015 98.179255)
 		(end 173.575015 102.889606)
@@
 	)
 	(gr_line
-		(start 168.610538 42.387003)
-		(end 170.091149 41.438502)
+		(start 181.9118 109.589594)
+		(end 181.9118 102.68275)
 		(stroke
 			(width 0.05)
-			(type default)
+			(type solid)
 		)
-		(locked yes)
 		(layer "Edge.Cuts")
 	)
-	(gr_arc
-		(start 207.609488 115.199839)
-		(mid 207.851876 115.262512)
-		(end 208.033488 115.434839)
+	(gr_line
+		(start 168.610538 42.387003)
+		(end 170.091149 41.438502)
 		(stroke
 			(width 0.05)
 			(type default)
 		)
+		(locked yes)
 		(layer "Edge.Cuts")
 	)
@@
 	)
 	(gr_line
+		(start 175.514 60.452)
+		(end 175.508508 66.052)
+		(stroke
+			(width 0.05)
+			(type default)
+		)
+		(layer "Edge.Cuts")
+	)
+	(gr_line
 		(start 169.524807 32.316)
 		(end 169.524807 37.026351)
@@
 		)
 	)
+	(gr_text "widened flexure to gain 0.6mm width"
+		(at 152.3 89.9 0)
+		(layer "Cmts.User")
+		(effects
+			(font
+				(size 1 1)
+				(thickness 0.1)
+			)
+			(justify left bottom)
+		)
+	)
 	(table
 		(column_count 2)
@@
 		)
 	)
+	(group ""
+		(members "2aca7457-a89a-45da-994c-84349ba58ca4" "4dfb9c3c-e017-4ba2-92f3-90506e1ef42f"
+			"b3ef76c8-0c8f-4f0f-ad14-6f486aef0107" "b49b2dd9-dbe0-41d8-9b5f-12298da8481a"
+			"b9314f11-8089-42a4-8420-0309d2b5f795" "c286579e-ec84-4dd3-ae30-f4de6ff13f7e"
+		)
+	)

Commit message: final save before duplication
saved draft in templates
Parts:
- removed the U201 at (171.8, 105.5)
- removed the U202 at (171.8, 119.2)
- added REF**: Throughhole_Motorshaft_7.5mm, ulib_Mechanical:Throughhole_Motorshaft_7.5mm, F.Cu at (188.0, 46.5)
- added REF**: MountingHole_2.9mm_M2.5, ulib_Mechanical:MountingHole_2.9mm_M2.5, F.Cu at (198.6, 52.4)
- added REF**: MountingHole_2.9mm_M2.5, ulib_Mechanical:MountingHole_2.9mm_M2.5, F.Cu at (177.3, 40.7)
Other:
- board size 95.7 x 97.3 mm -> 88.2 x 31.4 mm
- board text added: "optimiized neck at flexure for 0.068{dblquote} mill bit, widened flexure to gain 0.6mm width, inserted standoff architecture from mechanical"
- board text removed: "Widened channel between M2 and flexure to be exact mill bit dimensions of 0.068{dblquote} diameter"
- board text removed: "widened flexure to gain 0.6mm width"
