File: Strain Gauge POC Board V1/Single Bridge 1.kicad_sch (KiCad schematic)
At the start: 40 parts, among them J202 502352-0210, J203 502352-0210, U201 INA333xxDGK, U202 ADS1113IDGSR

Commit message: dev
Parts:
- removed FID201, FID202: Fiducial, ulib_Mechanical:Fiducial_0.5mm_Mask1mm, symbol ulib_Mounting_Holes:Fiducial
- renumbered C204 to C202, C205 to C204, J202 to J201, J203 to J202, R203 to R202, R202 to R203, R217 to R204, R218 to R207, R207 to R210, R204 to R213, R210 to R214, R213 to R215, R214 to R216, U203 to U201, U204 to U202, U209 to U203, U210 to U204, U201 to U209, U202 to U210
Changed lines of the file:
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@@
 		(dnp no)
 		(fields_autoplaced yes)
-		(property "Reference" "J203"
+		(property "Reference" "J202"
 			(at 528.32 206.3749 90)
 			(effects
@@
 			(project "Strain Gauge POC Board V1"
 				(path "/86d41315-8564-4bca-9150-9edda69acf24/c4515538-bae9-4cf8-b6d8-6ea87fa2c929"
-					(reference "J203")
+					(reference "J202")
 					(unit 1)
 				)
@@
 		(dnp no)
 		(fields_autoplaced yes)
-		(property "Reference" "U209"
+		(property "Reference" "U203"
 			(at 58.42 327.0249 0)
 			(effects
@@
 			(project "Strain Gauge POC Board V1"
 				(path "/86d41315-8564-4bca-9150-9edda69acf24/c4515538-bae9-4cf8-b6d8-6ea87fa2c929"
-					(reference "U209")
+					(reference "U203")
 					(unit 1)
 				)
@@
 	)
 	(symbol
-		(lib_id "ulib_Mounting_Holes:Fiducial")
-		(at 91.44 322.58 0)
-		(unit 1)
-		(exclude_from_sim no)
-		(in_bom yes)
-		(on_board yes)
-		(dnp no)
-		(fields_autoplaced yes)
-		(property "Reference" "FID202"
-			(at 93.98 321.3099 0)
-			(effects
-				(font
-					(size 1.27 1.27)
-				)
-				(justify left)
-			)
-		)
-		(property "Value" "Fiducial"
-			(at 93.98 323.8499 0)
-			(effects
-				(font
-					(size 1.27 1.27)
-				)
-				(justify left)
-			)
-		)
-		(property "Footprint" "ulib_Mechanical:Fiducial_0.5mm_Mask1mm"
-			(at 91.44 322.58 0)
-			(effects
-				(font
-					(size 1.27 1.27)
-				)
-				(hide yes)
-			)
-		)
-		(property "Datasheet" "~"
-			(at 91.44 322.58 0)
-			(effects
-				(font
-					(size 1.27 1.27)
-				)
-				(hide yes)
-			)
-		)
-		(property "Description" "Fiducial Marker"
-			(at 91.44 322.58 0)
-			(effects
-				(font
-					(size 1.27 1.27)
-				)
-				(hide yes)
-			)
-		)
-		(instances
-			(project "Strain Gauge POC Board V1"
-				(path "/86d41315-8564-4bca-9150-9edda69acf24/c4515538-bae9-4cf8-b6d8-6ea87fa2c929"
-					(reference "FID202")
-					(unit 1)
-				)
-			)
-		)
-	)
-	(symbol
 		(lib_id "power:GND")
 		(at 50.8 342.9 0)
@@
 		(on_board yes)
 		(dnp yes)
-		(property "Reference" "R214"
+		(property "Reference" "R216"
 			(at 543.56 205.1049 0)
 			(effects
@@
 			(project "Strain Gauge POC Board V1"
 				(path "/86d41315-8564-4bca-9150-9edda69acf24/c4515538-bae9-4cf8-b6d8-6ea87fa2c929"
-					(reference "R214")
+					(reference "R216")
 					(unit 1)
 				)
@@
 		(on_board yes)
 		(dnp no)
-		(property "Reference" "R203"
+		(property "Reference" "R202"
 			(at 238.76 169.5449 0)
 			(effects
@@
 			(project "Strain Gauge POC Board V1"
 				(path "/86d41315-8564-4bca-9150-9edda69acf24/c4515538-bae9-4cf8-b6d8-6ea87fa2c929"
-					(reference "R203")
+					(reference "R202")
 					(unit 1)
 				)
@@
 		(dnp yes)
 		(fields_autoplaced yes)
-		(property "Reference" "R202"
+		(property "Reference" "R203"
 			(at 238.76 230.5049 0)
 			(effects
@@
 			(project "Strain Gauge POC Board V1"
 				(path "/86d41315-8564-4bca-9150-9edda69acf24/c4515538-bae9-4cf8-b6d8-6ea87fa2c929"
-					(reference "R202")
+					(reference "R203")
 					(unit 1)
 				)
@@
 		(on_board yes)
 		(dnp no)
-		(property "Reference" "U201"
+		(property "Reference" "U209"
 			(at 317.246 196.342 0)
 			(effects
@@
 			(project "Strain Gauge POC Board V1"
 				(path "/86d41315-8564-4bca-9150-9edda69acf24/c4515538-bae9-4cf8-b6d8-6ea87fa2c929"
-					(reference "U201")
+					(reference "U209")
 					(unit 1)
 				)
@@
 		(on_board yes)
 		(dnp no)
-		(property "Reference" "J202"
+		(property "Reference" "J201"
 			(at 121.67 158.75 90)
 			(effects
@@
 			(project ""
 				(path "/86d41315-8564-4bca-9150-9edda69acf24/c4515538-bae9-4cf8-b6d8-6ea87fa2c929"
-					(reference "J202")
+					(reference "J201")
 					(unit 1)
 				)
@@
 		(dnp no)
 		(fields_autoplaced yes)
-		(property "Reference" "U204"
+		(property "Reference" "U202"
 			(at 58.42 316.8649 0)
 			(effects
@@
 			(project "Strain Gauge POC Board V1"
 				(path "/86d41315-8564-4bca-9150-9edda69acf24/c4515538-bae9-4cf8-b6d8-6ea87fa2c929"
-					(reference "U204")
+					(reference "U202")
 					(unit 1)
 				)
@@
 		(on_board yes)
 		(dnp no)
-		(property "Reference" "R210"
+		(property "Reference" "R214"
 			(at 500.38 189.8649 0)
 			(effects
@@
 			(project "Strain Gauge POC Board V1"
 				(path "/86d41315-8564-4bca-9150-9edda69acf24/c4515538-bae9-4cf8-b6d8-6ea87fa2c929"
-					(reference "R210")
+					(reference "R214")
 					(unit 1)
 				)
@@
 		(dnp no)
 		(fields_autoplaced yes)
-		(property "Reference" "U202"
+		(property "Reference" "U210"
 			(at 449.0086 190.5 0)
 			(effects
@@
 			(project ""
 				(path "/86d41315-8564-4bca-9150-9edda69acf24/c4515538-bae9-4cf8-b6d8-6ea87fa2c929"
-					(reference "U202")
+					(reference "U210")
 					(unit 1)
 				)
@@
 		(dnp no)
 		(fields_autoplaced yes)
-		(property "Reference" "U210"
+		(property "Reference" "U204"
 			(at 58.42 337.1849 0)
 			(effects
@@
 			(project "Strain Gauge POC Board V1"
 				(path "/86d41315-8564-4bca-9150-9edda69acf24/c4515538-bae9-4cf8-b6d8-6ea87fa2c929"
-					(reference "U210")
+					(reference "U204")
 					(unit 1)
 				)
@@
 		(on_board yes)
 		(dnp yes)
-		(property "Reference" "R213"
+		(property "Reference" "R215"
 			(at 502.92 210.1849 0)
 			(effects
@@
 			(project "Strain Gauge POC Board V1"
 				(path "/86d41315-8564-4bca-9150-9edda69acf24/c4515538-bae9-4cf8-b6d8-6ea87fa2c929"
-					(reference "R213")
+					(reference "R215")
 					(unit 1)
 				)
@@
 		(dnp no)
 		(fields_autoplaced yes)
-		(property "Reference" "C205"
+		(property "Reference" "C204"
 			(at 469.9 179.7049 0)
 			(effects
@@
 			(project ""
 				(path "/86d41315-8564-4bca-9150-9edda69acf24/c4515538-bae9-4cf8-b6d8-6ea87fa2c929"
-					(reference "C205")
+					(reference "C204")
 					(unit 1)
 				)
@@
 		(dnp no)
 		(fields_autoplaced yes)
-		(property "Reference" "C204"
+		(property "Reference" "C202"
 			(at 317.5 174.6249 0)
 			(effects
@@
 			(project "Strain Gauge POC Board V1"
 				(path "/86d41315-8564-4bca-9150-9edda69acf24/c4515538-bae9-4cf8-b6d8-6ea87fa2c929"
-					(reference "C204")
+					(reference "C202")
 					(unit 1)
 				)
@@
 		(on_board yes)
 		(dnp no)
-		(property "Reference" "R217"
+		(property "Reference" "R204"
 			(at 243.84 202.5649 0)
 			(effects
@@
 			(project "Strain Gauge POC Board V1"
 				(path "/86d41315-8564-4bca-9150-9edda69acf24/c4515538-bae9-4cf8-b6d8-6ea87fa2c929"
-					(reference "R217")
+					(reference "R204")
 					(unit 1)
 				)
@@
 		(on_board yes)
 		(dnp no)
-		(property "Reference" "R207"
+		(property "Reference" "R210"
 			(at 381.508 189.484 90)
 			(effects
@@
 			(project "Strain Gauge POC Board V1"
 				(path "/86d41315-8564-4bca-9150-9edda69acf24/c4515538-bae9-4cf8-b6d8-6ea87fa2c929"
-					(reference "R207")
+					(reference "R210")
 					(unit 1)
 				)
@@
 		(on_board yes)
 		(dnp no)
-		(property "Reference" "R218"
+		(property "Reference" "R207"
 			(at 297.18 197.4849 0)
 			(effects
@@
 			(project "Strain Gauge POC Board V1"
 				(path "/86d41315-8564-4bca-9150-9edda69acf24/c4515538-bae9-4cf8-b6d8-6ea87fa2c929"
-					(reference "R218")
+					(reference "R207")
 					(unit 1)
 				)
@@
 		(dnp no)
 		(fields_autoplaced yes)
-		(property "Reference" "U203"
+		(property "Reference" "U201"
 			(at 58.42 306.7049 0)
 			(effects
@@
 			(project ""
 				(path "/86d41315-8564-4bca-9150-9edda69acf24/c4515538-bae9-4cf8-b6d8-6ea87fa2c929"
-					(reference "U203")
-					(unit 1)
-				)
-			)
-		)
-	)
-	(symbol
-		(lib_id "ulib_Mounting_Holes:Fiducial")
-		(at 91.44 307.34 0)
-		(unit 1)
-		(exclude_from_sim no)
-		(in_bom yes)
-		(on_board yes)
-		(dnp no)
-		(fields_autoplaced yes)
-		(property "Reference" "FID201"
-			(at 93.98 306.0699 0)
-			(effects
-				(font
-					(size 1.27 1.27)
-				)
-				(justify left)
-			)
-		)
-		(property "Value" "Fiducial"
-			(at 93.98 308.6099 0)
-			(effects
-				(font
-					(size 1.27 1.27)
-				)
-				(justify left)
-			)
-		)
-		(property "Footprint" "ulib_Mechanical:Fiducial_0.5mm_Mask1mm"
-			(at 91.44 307.34 0)
-			(effects
-				(font
-					(size 1.27 1.27)
-				)
-				(hide yes)
-			)
-		)
-		(property "Datasheet" "~"
-			(at 91.44 307.34 0)
-			(effects
-				(font
-					(size 1.27 1.27)
-				)
-				(hide yes)
-			)
-		)
-		(property "Description" "Fiducial Marker"
-			(at 91.44 307.34 0)
-			(effects
-				(font
-					(size 1.27 1.27)
-				)
-				(hide yes)
-			)
-		)
-		(instances
-			(project ""
-				(path "/86d41315-8564-4bca-9150-9edda69acf24/c4515538-bae9-4cf8-b6d8-6ea87fa2c929"
-					(reference "FID201")
+					(reference "U201")
 					(unit 1)
 				)
@@
 		(on_board yes)
 		(dnp no)
-		(property "Reference" "R204"
+		(property "Reference" "R213"
 			(at 485.14 189.8649 0)
 			(effects
@@
 			(project "Strain Gauge POC Board V1"
 				(path "/86d41315-8564-4bca-9150-9edda69acf24/c4515538-bae9-4cf8-b6d8-6ea87fa2c929"
-					(reference "R204")
+					(reference "R213")
 					(unit 1)
 				)

Commit message: bulk of first draft done
Parts:
- added FID201, FID202, FID203, FID204: Fiducial, ulib_Mechanical:Fiducial_0.5mm_Mask1mm, symbol ulib_Mounting_Holes:Fiducial

Commit message: Ready for fab sans watermark
Connections:
- net +3V3a: now also R216.2; no longer R216.1
- net GND: no longer U201.MP, U202.MP, U203.MP, U204.MP
- net ADC_I2C_SDA: now reaches J202.1, R213.2, U210.9 (SDA)
- net ADC_I2C_SDA: now also R212.2; no longer R212.1
- net ADC_I2C_SCL: now reaches J202.2, R214.2, U210.10 (SCL)
- net ADC_I2C_SCL: now also R215.2; no longer R215.1
- net at R202.2, R204.1, R205.2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: now also R203.1
- new net: R211.1, R212.1, R215.1, R216.1, U210.1 (ADDR)
- no-connect marks 0 -> 4
Other:
- note added: "Address configuration resistors"
- moved on the sheet: C201, C202, C203, C204, FID201, FID202, FID203, FID204, J201, J202, R201, R202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
