File: Strain Gauge POC Board V1/Strain Gauge POC Board V1/Single Bridge 1.kicad_sch (KiCad schematic)
At the start: 42 parts, among them J201 502352-0210, J202 502352-0210, U209 INA333xxDGK, U210 ADS1113IDGSR

Commit message: dev
Parts:
- renumbered C201 to C1, C202 to C2, C203 to C3, C204 to C4, FID201 to FID1, FID202 to FID2, FID203 to FID3, FID204 to FID4, J201 to J1, J202 to J2, R201 to R1, R210 to R10, R213 to R11, R211 to R12, R212 to R13, R214 to R14, R215 to R15, R216 to R16, R203 to R2, R202 to R3, R204 to R4, R205 to R5, R206 to R6, R207 to R7, R208 to R8, R209 to R9, TP201 to TP1, TP202 to TP2, TP203 to TP3, TP204 to TP4, TP205 to TP5, TP206 to TP6, U201 to U1, U210 to U10, U202 to U2, U203 to U3, U204 to U4, U205 to U5, U206 to U6, U207 to U7, U208 to U8, U209 to U9

Commit message: ready for fab
Connections:
- net +3V3a renamed +3V3
Changed lines of the file:
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@@
 			)
 		)
-		(property "Value" "+3V3a"
+		(property "Value" "+3V3"
 			(at 459.74 165.1 0)
 			(effects
@@
 			)
 		)
-		(property "Value" "+3V3a"
+		(property "Value" "+3V3"
 			(at 162.56 154.94 0)
 			(effects
@@
 			)
 		)
-		(property "Value" "+3V3a"
+		(property "Value" "+3V3"
 			(at 322.58 165.1 0)
 			(effects
@@
 			)
 		)
-		(property "Value" "+3V3a"
+		(property "Value" "+3V3"
 			(at 370.84 205.74 0)
 			(effects
@@
 			)
 		)
-		(property "Value" "+3V3a"
+		(property "Value" "+3V3"
 			(at 45.72 149.86 0)
 			(effects
@@
 			)
 		)
-		(property "Value" "+3V3a"
+		(property "Value" "+3V3"
 			(at 548.64 241.3 0)
 			(effects
