File: Strain Gauge POC Board V1/Strain Gauge POC Board V1/Strain Gauge POC Board V1.kicad_pcb (KiCad board)
At the start: 4 copper layers, 88.2 x 31.4 mm, 46 parts, among them J201 502352-0210, J202 502352-0210, U209 INA333xxDGK, U210 ADS1113IDGSR

Commit message: dev
Parts:
- moved R13 51.5 mm to (144.0, 101.6)
- moved C3 51.5 mm to (149.9, 98.7)
- moved U9 51.5 mm to (155.9, 97.5)
- moved FID1 51.5 mm to (111.3, 91.4)
- moved FID2 51.5 mm to (157.0, 86.3)
- moved J2 51.5 mm to (117.7, 107.9)
- moved R12 51.5 mm to (147.3, 101.6)
- moved R15 51.5 mm to (142.4, 101.6)
- moved R16 51.5 mm to (145.7, 101.6)
- moved R7 51.5 mm to (156.0, 100.3)
- moved C1 51.5 mm to (154.3, 104.4)
- moved C4 51.5 mm to (141.1, 95.4)
- moved FID3 51.5 mm to (111.3, 111.0)
- moved FID4 51.5 mm to (157.2, 111.0)
- moved G*** 51.5 mm to (123.2, 86.6)
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- renumbered C201 to C1, C202 to C2, C203 to C3, C204 to C4, FID201 to FID1, FID202 to FID2, FID203 to FID3, FID204 to FID4, J201 to J1, J202 to J2, R201 to R1, R210 to R10, R213 to R11, R211 to R12, R212 to R13, R214 to R14, R215 to R15, R216 to R16, R203 to R2, R202 to R3, R204 to R4, R205 to R5, R206 to R6, R207 to R7, R208 to R8, R209 to R9, TP201 to TP1, TP202 to TP2, TP203 to TP3, TP204 to TP4, TP205 to TP5, TP206 to TP6, U201 to U1, U210 to U10, U202 to U2, U203 to U3, U204 to U4, U205 to U5, U206 to U6, U207 to U7, U208 to U8, U209 to U9
Routing:
- net Net-(U9-+): track 132.2 -> 149.3 mm
Other:
- board size 88.2 x 31.4 mm -> 89.2 x 31.4 mm

Commit message: ready for fab
Parts:
- moved U4 0.39 mm to (131.3, 104.5)
- moved U3 0.36 mm to (131.3, 90.8)
Connections:
- net +3V3a renamed +3V3
Routing:
- net Net-(U9-+): track 149.3 -> 180.2 mm
Other:
- outline, holes or cut-outs redrawn

Commit message: ready for fab for real this time
Routing:
- net Net-(U9-+): track 180.2 -> 189.9 mm
